File: PCB Layout/kicad/LightMeter_MegaShield.kicad_pcb (KiCad board)
At the start: 2 copper layers, 90.6 x 102 mm, 49 parts, among them J1 microSD DM3AT-SF-PEJM5, J10 LUX2 TSL2591, J11 ENCODER, J2 LCD 20x4 I2C, J3 LUX1 TSL2591, J4 LED1 GPS, J5 LED2 LUX, J6 LED3 IMU, J7 BTN SLEEP, J8 BTN LOG TOGGLE, J9 BTN FORCE LOG, U1 74LVC125A, U2 AMS1117-3.3, U3 PCA9548AD (SOIC-24W)

Commit message: PCB Layout: fix status-LED wiring for common-cathode LEDs, validation pass
- LED connectors J4-J6: pin 1 is now GND (common cathode) and each *_red pin
  drives the red die, matching setLED() in the Week 5-8 sketches
  (HIGH = on, YELLOW = both HIGH). The old 5V/common-anode wiring would
  have swapped YELLOW and OFF with Week 8.
  GPS red D4 / green D7, LUX red D5 / green D6, IMU red D8 / green D9.
- Rerouted; silkscreen now reads "GND R G"; Gerbers, drills, BOM, renders,
  schematic PDF and STEP regenerated. ERC 0, DRC 0, parity 0.
- README: IMU orientation matters (Week 8 checks roll only), header
  trimming applies to GPS/IMU pins only, updated counts and boot sequence.
- Verified GPS/BNO055 footprints against Adafruit board files and the Mega
  footprint pad-by-pad against KiCad's Arduino Mega template.

Co-Authored-By: Claude Opus 5.5 <noreply@anthropic.com>
Connections:
- A1 pad D4: LED1_G_MCU -> LED1_R_MCU
- A1 pad D5: LED2_G_MCU -> LED2_R_MCU
- A1 pad D6: LED2_R_MCU -> LED2_G_MCU
- A1 pad D7: LED1_R_MCU -> LED1_G_MCU
- A1 pad D8: LED3_G_MCU -> LED3_R_MCU
- A1 pad D9: LED3_R_MCU -> LED3_G_MCU
- J4 pad 1: +5V -> GND
- J5 pad 1: +5V -> GND
- J6 pad 1: +5V -> GND
Routing:
- net GND: track 439.3 -> 530.3 mm, vias 3 -> 0
- net LED1_R_MCU: track 70.0 -> 50.3 mm, vias 1 -> 0
- net LED1_R: track 81.5 -> 64.9 mm, vias 1 -> 0
- net BTN_LOG: track 116.8 -> 130.2 mm, vias 3 -> 1
- net GPS_TX: track 92.3 -> 102.5 mm
- net IMU_3V3: track 23.6 -> 33.1 mm
- net +3V3: track 77.7 -> 87.0 mm, vias 4 -> 5
- net SPI_MOSI: track 65.5 -> 74.7 mm
- net LED1_G_MCU: track 46.8 -> 56.0 mm, vias 0 -> 1
- net SCL: track 153.9 -> 146.3 mm
- net ENC_A: track 18.2 -> 25.4 mm, vias 0 -> 1
- net ENC_A_MCU: track 50.3 -> 43.3 mm, vias 2 -> 0
- net IMU_TX: track 37.2 -> 30.4 mm, vias 1 -> 0
- net LED3_R_MCU: track 66.1 -> 59.9 mm
- net SPI_MISO: track 87.9 -> 81.9 mm, vias 0 -> 2
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Other:
- board text added: "ARDUINO MEGA 2560 PLUGS IN HERE"
- board text added: "GPS LED GND R G"
- board text added: "IMU LED GND R G"
- board text added: "LUX LED GND R G"
- board text removed: "ARDUINO MEGA 2560 PLUGS IN HERE (stacking headers)"
- board text removed: "LED1 GPS 5V R G"
- board text removed: "LED2 LUX 5V R G"
- board text removed: "LED3 IMU 5V R G"

Commit message: PCB Layout: assembly validation fixes
- C5 bulk cap: 6.3 mm / 2.5 mm-pitch footprint (0.9 mm pad gap instead of
  0.4 mm between +5V and GND), moved clear of J9
- microSD card-detect pad 9 left unconnected (0.25 mm from DAT1, a solder
  bridge there is now harmless)
- no tracks/vias under screw heads and standoffs at every mounting hole;
  rerouted, ERC 0, DRC 0, parity 0, Gerbers/drills/zip regenerated
- README: buy list, cable pinouts, LED/button mis-plug warning, GPS
  standoff method for the coin-cell holder, corrected power budget

Co-Authored-By: Claude Opus 5.5 <noreply@anthropic.com>
Parts:
- C5: footprint Capacitor_THT:CP_Radial_D5.0mm_P2.00mm -> Capacitor_THT:CP_Radial_D6.3mm_P2.50mm
- moved C5 2.20 mm to (48.0, -84.2)
Connections:
- J1 pad 9: GND -> unconnected-(J1-DET_B-Pad9)
Routing:
- net +5V: track 387.0 -> 354.1 mm, vias 1 -> 3
- net GND: track 530.3 -> 504.2 mm, vias 0 -> 1
- net LED1_R_MCU: track 50.3 -> 73.3 mm, vias 0 -> 1
- net SDA: track 126.3 -> 148.9 mm, vias 4 -> 2
- net IMU_PS1: track 67.1 -> 89.3 mm, vias 4 -> 1
- net LED1_R: track 64.9 -> 85.2 mm, vias 0 -> 1
- net ENC_B_MCU: track 48.1 -> 61.5 mm, vias 2 -> 0
- net LED2_G: track 48.4 -> 60.8 mm
- net SD_CLK: track 25.4 -> 13.8 mm
- net IMU_TX: track 30.4 -> 41.5 mm, vias 0 -> 2
- net LED1_G_MCU: track 56.0 -> 66.1 mm
- net SPI_MOSI: track 74.7 -> 65.0 mm
- net ENC_A: track 25.4 -> 17.0 mm
- net GPS_TX: track 102.5 -> 94.7 mm
- net LED3_R_MCU: track 59.9 -> 52.9 mm
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