File: PCB Layout/kicad/LightMeter_MegaShield.kicad_sch (KiCad schematic)
At the start: 49 parts, among them J1 microSD DM3AT-SF-PEJM5, J10 LUX2 TSL2591, J11 ENCODER, J2 LCD 20x4 I2C, J3 LUX1 TSL2591, J4 LED1 GPS, J5 LED2 LUX, J6 LED3 IMU, J7 BTN SLEEP, J8 BTN LOG TOGGLE, J9 BTN FORCE LOG, U1 74LVC125A, U2 AMS1117-3.3, U3 PCA9548AD (SOIC-24W)

Commit message: PCB Layout: fix status-LED wiring for common-cathode LEDs, validation pass
- LED connectors J4-J6: pin 1 is now GND (common cathode) and each *_red pin
  drives the red die, matching setLED() in the Week 5-8 sketches
  (HIGH = on, YELLOW = both HIGH). The old 5V/common-anode wiring would
  have swapped YELLOW and OFF with Week 8.
  GPS red D4 / green D7, LUX red D5 / green D6, IMU red D8 / green D9.
- Rerouted; silkscreen now reads "GND R G"; Gerbers, drills, BOM, renders,
  schematic PDF and STEP regenerated. ERC 0, DRC 0, parity 0.
- README: IMU orientation matters (Week 8 checks roll only), header
  trimming applies to GPS/IMU pins only, updated counts and boot sequence.
- Verified GPS/BNO055 footprints against Adafruit board files and the Mega
  footprint pad-by-pad against KiCad's Arduino Mega template.

Co-Authored-By: Claude Opus 5.5 <noreply@anthropic.com>
Connections:
- net +5V: no longer J4.1 (Pin_1), J5.1 (Pin_1), J6.1 (Pin_1)
- net GND: now also J4.1 (Pin_1), J5.1 (Pin_1), J6.1 (Pin_1)
- net LED1_G_MCU: now also A1.D7; no longer A1.D4
- net LED1_R_MCU: now also A1.D4; no longer A1.D7
- net LED2_G_MCU: now also A1.D6; no longer A1.D5
- net LED2_R_MCU: now also A1.D5; no longer A1.D6
- net LED3_G_MCU: now also A1.D9; no longer A1.D8
- net LED3_R_MCU: now also A1.D8; no longer A1.D9
Other:
- note added: "Connector pinouts (JST-XH): LCD/LUX = GND,5V,SDA,SCL LEDx = GND(common cathode),RED,GREEN BTNx = GND,SW,5V(lamp)"
- note added: "Pin map from the team sketch (Lightmeter_Week8.ino): SD CS=D53 (HW SPI 50/51/52), GPS=Serial1 (D18/D19), IMU=Serial2 (D16/D17), I2C=D20/D21, LEDs common-cathode to GND, active HIGH (setLED() in Week 5-8 sketches: YELLOW = both HIGH): GPS R=D4 G=D7, LUX R=D5 G=D6, IMU R=D8 G=D9; buttons to GND with INPUT_PULLUP: sleep D10, log toggle D11, force log D12."
- note removed: "Connector pinouts (JST-XH): LCD/LUX = GND,5V,SDA,SCL LEDx = 5V(common anode),RED,GREEN BTNx = GND,SW,5V(lamp)"
- note removed: "Pin map from latest_version_of_lightmeter.ino: SD CS=D53 (HW SPI 50/51/52), GPS=Serial1 (D18/D19), IMU=Serial2 (D16/D17), I2C=D20/D21, LEDs common-anode to 5V, active LOW. setLED(GREEN) pulls the *_red pin LOW, so *_red pins drive the GREEN die: GPS G=D4 R=D7, LUX G=D5 R=D6, IMU G=D8 R=D9, LUX D5/D6, IMU D8/D9; buttons to GND with INPUT_PULLUP: sleep D10, log toggle D11, force log D12."

Commit message: PCB Layout: assembly validation fixes
- C5 bulk cap: 6.3 mm / 2.5 mm-pitch footprint (0.9 mm pad gap instead of
  0.4 mm between +5V and GND), moved clear of J9
- microSD card-detect pad 9 left unconnected (0.25 mm from DAT1, a solder
  bridge there is now harmless)
- no tracks/vias under screw heads and standoffs at every mounting hole;
  rerouted, ERC 0, DRC 0, parity 0, Gerbers/drills/zip regenerated
- README: buy list, cable pinouts, LED/button mis-plug warning, GPS
  standoff method for the coin-cell holder, corrected power budget

Co-Authored-By: Claude Opus 5.5 <noreply@anthropic.com>
Parts:
- C5: footprint Capacitor_THT:CP_Radial_D5.0mm_P2.00mm -> Capacitor_THT:CP_Radial_D6.3mm_P2.50mm
Connections:
- net GND: no longer J1.9 (DET_B)
- no-connect marks 87 -> 88
